Commit message: Sucessfuly changed the urdf

File: assets/nmf_no_limits.urdf (robot description, URDF)
Before this commit: robot neuromechfly_noLimits, 93 links, 92 joints
Links:
- link A1A2: geometry collision mesh filename=/home/achard/stlfiles/A1A2.stl scale=1000.0 1000.0 1000.0; visual mesh filename=/home/achard/stlfiles/A1A2.stl scale=1000.0 1000.0 1000.0
- link A3: geometry collision mesh filename=/home/achard/stlfiles/A3.stl scale=1000.0 1000.0 1000.0; visual mesh filename=/home/achard/stlfiles/A3.stl scale=1000.0 1000.0 1000.0
- link A4: geometry collision mesh filename=/home/achard/stlfiles/A4.stl scale=1000.0 1000.0 1000.0; visual mesh filename=/home/achard/stlfiles/A4.stl scale=1000.0 1000.0 1000.0
- link A5: geometry collision mesh filename=/home/achard/stlfiles/A5.stl scale=1000.0 1000.0 1000.0; visual mesh filename=/home/achard/stlfiles/A5.stl scale=1000.0 1000.0 1000.0
- link A6: geometry collision mesh filename=/home/achard/stlfiles/A6.stl scale=1000.0 1000.0 1000.0; visual mesh filename=/home/achard/stlfiles/A6.stl scale=1000.0 1000.0 1000.0
- link Haustellum: geometry collision mesh filename=/home/achard/stlfiles/Haustellum.stl scale=1000.0 1000.0 1000.0; visual mesh filename=/home/achard/stlfiles/Haustellum.stl scale=1000.0 1000.0 1000.0
- link Head: geometry collision mesh filename=/home/achard/stlfiles/Head.stl scale=1000.0 1000.0 1000.0; visual mesh filename=/home/achard/stlfiles/Head.stl scale=1000.0 1000.0 1000.0
- link LAntenna: geometry collision mesh filename=/home/achard/stlfiles/LAntenna.stl scale=1000.0 1000.0 1000.0; visual mesh filename=/home/achard/stlfiles/LAntenna.stl scale=1000.0 1000.0 1000.0
- link LEye: geometry collision mesh filename=/home/achard/stlfiles/LEye.stl scale=1000.0 1000.0 1000.0; visual mesh filename=/home/achard/stlfiles/LEye.stl scale=1000.0 1000.0 1000.0
- link LFCoxa: geometry collision mesh filename=/home/achard/stlfiles/LFCoxa.stl scale=1000.0 1000.0 1000.0; visual mesh filename=/home/achard/stlfiles/LFCoxa.stl scale=1000.0 1000.0 1000.0
- link LFFemur: geometry collision mesh filename=/home/achard/stlfiles/LFFemur.stl scale=1000.0 1000.0 1000.0; visual mesh filename=/home/achard/stlfiles/LFFemur.stl scale=1000.0 1000.0 1000.0
- link LFTarsus1: geometry collision mesh filename=/home/achard/stlfiles/LFTarsus1.stl scale=1000.0 1000.0 1000.0; visual mesh filename=/home/achard/stlfiles/LFTarsus1.stl scale=1000.0 1000.0 1000.0
- link LFTarsus2: geometry collision mesh filename=/home/achard/stlfiles/LFTarsus2.stl scale=1000.0 1000.0 1000.0; visual mesh filename=/home/achard/stlfiles/LFTarsus2.stl scale=1000.0 1000.0 1000.0
- link LFTarsus3: geometry collision mesh filename=/home/achard/stlfiles/LFTarsus3.stl scale=1000.0 1000.0 1000.0; visual mesh filename=/home/achard/stlfiles/LFTarsus3.stl scale=1000.0 1000.0 1000.0
- link LFTarsus4: geometry collision mesh filename=/home/achard/stlfiles/LFTarsus4.stl scale=1000.0 1000.0 1000.0; visual mesh filename=/home/achard/stlfiles/LFTarsus4.stl scale=1000.0 1000.0 1000.0
- link LFTarsus5: geometry collision mesh filename=/home/achard/stlfiles/LFTarsus5.stl scale=1000.0 1000.0 1000.0; visual mesh filename=/home/achard/stlfiles/LFTarsus5.stl scale=1000.0 1000.0 1000.0
- link LFTibia: geometry collision mesh filename=/home/achard/stlfiles/LFTibia.stl scale=1000.0 1000.0 1000.0; visual mesh filename=/home/achard/stlfiles/LFTibia.stl scale=1000.0 1000.0 1000.0
- link LHCoxa: geometry collision mesh filename=/home/achard/stlfiles/LHCoxa.stl scale=1000.0 1000.0 1000.0; visual mesh filename=/home/achard/stlfiles/LHCoxa.stl scale=1000.0 1000.0 1000.0
- link LHFemur: geometry collision mesh filename=/home/achard/stlfiles/LHFemur.stl scale=1000.0 1000.0 1000.0; visual mesh filename=/home/achard/stlfiles/LHFemur.stl scale=1000.0 1000.0 1000.0
- link LHTarsus1: geometry collision mesh filename=/home/achard/stlfiles/LHTarsus1.stl scale=1000.0 1000.0 1000.0; visual mesh filename=/home/achard/stlfiles/LHTarsus1.stl scale=1000.0 1000.0 1000.0
- link LHTarsus2: geometry collision mesh filename=/home/achard/stlfiles/LHTarsus2.stl scale=1000.0 1000.0 1000.0; visual mesh filename=/home/achard/stlfiles/LHTarsus2.stl scale=1000.0 1000.0 1000.0
- link LHTarsus3: geometry collision mesh filename=/home/achard/stlfiles/LHTarsus3.stl scale=1000.0 1000.0 1000.0; visual mesh filename=/home/achard/stlfiles/LHTarsus3.stl scale=1000.0 1000.0 1000.0
- link LHTarsus4: geometry collision mesh filename=/home/achard/stlfiles/LHTarsus4.stl scale=1000.0 1000.0 1000.0; visual mesh filename=/home/achard/stlfiles/LHTarsus4.stl scale=1000.0 1000.0 1000.0
- link LHTarsus5: geometry collision mesh filename=/home/achard/stlfiles/LHTarsus5.stl scale=1000.0 1000.0 1000.0; visual mesh filename=/home/achard/stlfiles/LHTarsus5.stl scale=1000.0 1000.0 1000.0
- link LHTibia: geometry collision mesh filename=/home/achard/stlfiles/LHTibia.stl scale=1000.0 1000.0 1000.0; visual mesh filename=/home/achard/stlfiles/LHTibia.stl scale=1000.0 1000.0 1000.0
- link LHaltere: geometry collision mesh filename=/home/achard/stlfiles/LHaltere.stl scale=1000.0 1000.0 1000.0; visual mesh filename=/home/achard/stlfiles/LHaltere.stl scale=1000.0 1000.0 1000.0
- link LMCoxa: geometry collision mesh filename=/home/achard/stlfiles/LMCoxa.stl scale=1000.0 1000.0 1000.0; visual mesh filename=/home/achard/stlfiles/LMCoxa.stl scale=1000.0 1000.0 1000.0
- link LMFemur: geometry collision mesh filename=/home/achard/stlfiles/LMFemur.stl scale=1000.0 1000.0 1000.0; visual mesh filename=/home/achard/stlfiles/LMFemur.stl scale=1000.0 1000.0 1000.0
- link LMTarsus1: geometry collision mesh filename=/home/achard/stlfiles/LMTarsus1.stl scale=1000.0 1000.0 1000.0; visual mesh filename=/home/achard/stlfiles/LMTarsus1.stl scale=1000.0 1000.0 1000.0
- link LMTarsus2: geometry collision mesh filename=/home/achard/stlfiles/LMTarsus2.stl scale=1000.0 1000.0 1000.0; visual mesh filename=/home/achard/stlfiles/LMTarsus2.stl scale=1000.0 1000.0 1000.0
- link LMTarsus3: geometry collision mesh filename=/home/achard/stlfiles/LMTarsus3.stl scale=1000.0 1000.0 1000.0; visual mesh filename=/home/achard/stlfiles/LMTarsus3.stl scale=1000.0 1000.0 1000.0
- link LMTarsus4: geometry collision mesh filename=/home/achard/stlfiles/LMTarsus4.stl scale=1000.0 1000.0 1000.0; visual mesh filename=/home/achard/stlfiles/LMTarsus4.stl scale=1000.0 1000.0 1000.0
- link LMTarsus5: geometry collision mesh filename=/home/achard/stlfiles/LMTarsus5.stl scale=1000.0 1000.0 1000.0; visual mesh filename=/home/achard/stlfiles/LMTarsus5.stl scale=1000.0 1000.0 1000.0
- link LMTibia: geometry collision mesh filename=/home/achard/stlfiles/LMTibia.stl scale=1000.0 1000.0 1000.0; visual mesh filename=/home/achard/stlfiles/LMTibia.stl scale=1000.0 1000.0 1000.0
- link LWing: geometry collision mesh filename=/home/achard/stlfiles/LWing.stl scale=1000.0 1000.0 1000.0; visual mesh filename=/home/achard/stlfiles/LWing.stl scale=1000.0 1000.0 1000.0
- link RAntenna: geometry collision mesh filename=/home/achard/stlfiles/RAntenna.stl scale=1000.0 1000.0 1000.0; visual mesh filename=/home/achard/stlfiles/RAntenna.stl scale=1000.0 1000.0 1000.0
- link REye: geometry collision mesh filename=/home/achard/stlfiles/REye.stl scale=1000.0 1000.0 1000.0; visual mesh filename=/home/achard/stlfiles/REye.stl scale=1000.0 1000.0 1000.0
- link RFCoxa: geometry collision mesh filename=/home/achard/stlfiles/RFCoxa.stl scale=1000.0 1000.0 1000.0; visual mesh filename=/home/achard/stlfiles/RFCoxa.stl scale=1000.0 1000.0 1000.0
- link RFFemur: geometry collision mesh filename=/home/achard/stlfiles/RFFemur.stl scale=1000.0 1000.0 1000.0; visual mesh filename=/home/achard/stlfiles/RFFemur.stl scale=1000.0 1000.0 1000.0
- link RFTarsus1: geometry collision mesh filename=/home/achard/stlfiles/RFTarsus1.stl scale=1000.0 1000.0 1000.0; visual mesh filename=/home/achard/stlfiles/RFTarsus1.stl scale=1000.0 1000.0 1000.0
- link RFTarsus2: geometry collision mesh filename=/home/achard/stlfiles/RFTarsus2.stl scale=1000.0 1000.0 1000.0; visual mesh filename=/home/achard/stlfiles/RFTarsus2.stl scale=1000.0 1000.0 1000.0
- link RFTarsus3: geometry collision mesh filename=/home/achard/stlfiles/RFTarsus3.stl scale=1000.0 1000.0 1000.0; visual mesh filename=/home/achard/stlfiles/RFTarsus3.stl scale=1000.0 1000.0 1000.0
- link RFTarsus4: geometry collision mesh filename=/home/achard/stlfiles/RFTarsus4.stl scale=1000.0 1000.0 1000.0; visual mesh filename=/home/achard/stlfiles/RFTarsus4.stl scale=1000.0 1000.0 1000.0
- link RFTarsus5: geometry collision mesh filename=/home/achard/stlfiles/RFTarsus5.stl scale=1000.0 1000.0 1000.0; visual mesh filename=/home/achard/stlfiles/RFTarsus5.stl scale=1000.0 1000.0 1000.0
- link RFTibia: geometry collision mesh filename=/home/achard/stlfiles/RFTibia.stl scale=1000.0 1000.0 1000.0; visual mesh filename=/home/achard/stlfiles/RFTibia.stl scale=1000.0 1000.0 1000.0
- link RHCoxa: geometry collision mesh filename=/home/achard/stlfiles/RHCoxa.stl scale=1000.0 1000.0 1000.0; visual mesh filename=/home/achard/stlfiles/RHCoxa.stl scale=1000.0 1000.0 1000.0
- link RHFemur: geometry collision mesh filename=/home/achard/stlfiles/RHFemur.stl scale=1000.0 1000.0 1000.0; visual mesh filename=/home/achard/stlfiles/RHFemur.stl scale=1000.0 1000.0 1000.0
- link RHTarsus1: geometry collision mesh filename=/home/achard/stlfiles/RHTarsus1.stl scale=1000.0 1000.0 1000.0; visual mesh filename=/home/achard/stlfiles/RHTarsus1.stl scale=1000.0 1000.0 1000.0
- link RHTarsus2: geometry collision mesh filename=/home/achard/stlfiles/RHTarsus2.stl scale=1000.0 1000.0 1000.0; visual mesh filename=/home/achard/stlfiles/RHTarsus2.stl scale=1000.0 1000.0 1000.0
- link RHTarsus3: geometry collision mesh filename=/home/achard/stlfiles/RHTarsus3.stl scale=1000.0 1000.0 1000.0; visual mesh filename=/home/achard/stlfiles/RHTarsus3.stl scale=1000.0 1000.0 1000.0
- link RHTarsus4: geometry collision mesh filename=/home/achard/stlfiles/RHTarsus4.stl scale=1000.0 1000.0 1000.0; visual mesh filename=/home/achard/stlfiles/RHTarsus4.stl scale=1000.0 1000.0 1000.0
- link RHTarsus5: geometry collision mesh filename=/home/achard/stlfiles/RHTarsus5.stl scale=1000.0 1000.0 1000.0; visual mesh filename=/home/achard/stlfiles/RHTarsus5.stl scale=1000.0 1000.0 1000.0
- link RHTibia: geometry collision mesh filename=/home/achard/stlfiles/RHTibia.stl scale=1000.0 1000.0 1000.0; visual mesh filename=/home/achard/stlfiles/RHTibia.stl scale=1000.0 1000.0 1000.0
- link RHaltere: geometry collision mesh filename=/home/achard/stlfiles/RHaltere.stl scale=1000.0 1000.0 1000.0; visual mesh filename=/home/achard/stlfiles/RHaltere.stl scale=1000.0 1000.0 1000.0
- link RMCoxa: geometry collision mesh filename=/home/achard/stlfiles/RMCoxa.stl scale=1000.0 1000.0 1000.0; visual mesh filename=/home/achard/stlfiles/RMCoxa.stl scale=1000.0 1000.0 1000.0
- link RMFemur: geometry collision mesh filename=/home/achard/stlfiles/RMFemur.stl scale=1000.0 1000.0 1000.0; visual mesh filename=/home/achard/stlfiles/RMFemur.stl scale=1000.0 1000.0 1000.0
- link RMTarsus1: geometry collision mesh filename=/home/achard/stlfiles/RMTarsus1.stl scale=1000.0 1000.0 1000.0; visual mesh filename=/home/achard/stlfiles/RMTarsus1.stl scale=1000.0 1000.0 1000.0
- link RMTarsus2: geometry collision mesh filename=/home/achard/stlfiles/RMTarsus2.stl scale=1000.0 1000.0 1000.0; visual mesh filename=/home/achard/stlfiles/RMTarsus2.stl scale=1000.0 1000.0 1000.0
- link RMTarsus3: geometry collision mesh filename=/home/achard/stlfiles/RMTarsus3.stl scale=1000.0 1000.0 1000.0; visual mesh filename=/home/achard/stlfiles/RMTarsus3.stl scale=1000.0 1000.0 1000.0
- link RMTarsus4: geometry collision mesh filename=/home/achard/stlfiles/RMTarsus4.stl scale=1000.0 1000.0 1000.0; visual mesh filename=/home/achard/stlfiles/RMTarsus4.stl scale=1000.0 1000.0 1000.0
- link RMTarsus5: geometry collision mesh filename=/home/achard/stlfiles/RMTarsus5.stl scale=1000.0 1000.0 1000.0; visual mesh filename=/home/achard/stlfiles/RMTarsus5.stl scale=1000.0 1000.0 1000.0
- link RMTibia: geometry collision mesh filename=/home/achard/stlfiles/RMTibia.stl scale=1000.0 1000.0 1000.0; visual mesh filename=/home/achard/stlfiles/RMTibia.stl scale=1000.0 1000.0 1000.0
- link RWing: geometry collision mesh filename=/home/achard/stlfiles/RWing.stl scale=1000.0 1000.0 1000.0; visual mesh filename=/home/achard/stlfiles/RWing.stl scale=1000.0 1000.0 1000.0
- link Rostrum: geometry collision mesh filename=/home/achard/stlfiles/Rostrum.stl scale=1000.0 1000.0 1000.0; visual mesh filename=/home/achard/stlfiles/Rostrum.stl scale=1000.0 1000.0 1000.0
- link Thorax: geometry collision mesh filename=/home/achard/stlfiles/Thorax.stl scale=1000.0 1000.0 1000.0; visual mesh filename=/home/achard/stlfiles/Thorax.stl scale=1000.0 1000.0 1000.0
Joints:
- joint joint_RHTarsus1: origin xyz=-2.6000e-04  6.6000e-04 -6.8445e-01 rpy=0 0 0 -> xyz=-2.6000e-04  6.6000e-04 -6.8445e-01 rpy=1 0 0
